File: MKRMotorCarrierV3.0/MKRMotorCarrierV3.0.brd (EAGLE design)
At the start: 53 x 80 mm, 20 parts, among them Q1 AON7407, Q3 AON7407, U1 DRV8871, U2 TS30013, U3 AH1815, X8 OSTTE/4

Commit message: Continued adding parts
Parts:
- removed U1: DRV8871, MKRMotorCarrierV3.0:SOIC127P600X170-8N
- removed U3: AH1815, MKRMotorCarrierV3.0:SIP3
Connections:
- removed net VCC: U3.1
- net GND: no longer U3.2
